File: hardware/cartridge/cartridge.kicad_pcb (KiCad board)
At the start: 2 copper layers, 71.2 x 52.2 mm, 31 parts, among them U1 SN74LVC8T245PWR, U2 SN74LVC8T245PWR, U3 SN74LVC8T245PWR, U4 SN74LVC8T245PWR, U5 LCMXO2-1200HC-4TG100C, U6 MX29LV320EBTI-70G, U7 FM28V100-TG, U8 RP2040-Zero

Commit message: Update schematics
Parts:
- added R3: 10K, Resistor_SMD:R_0603_1608Metric_Pad0.98x0.95mm_HandSolder, F.Cu at (161.2, 49.6)
Connections:
- U3 pad 22: Net-(U3-*OE) -> data_oe_n
- U5 pad 58: +3.3V -> data_oe_n
- U5 pad 96: unconnected-(U5-PT10B-Pad96) -> /SPI_MOSI
- U5 pad 97: unconnected-(U5-PT10A-Pad97) -> /SPI_CS_N
- U5 pad 98: unconnected-(U5-PT9B-Pad98) -> /SPI_SCK
- U5 pad 99: unconnected-(U5-PT9A-Pad99) -> /SPI_MISO
- U8 pad 0: unconnected-(U8-Pad0) -> /SPI_MISO
- U8 pad 1: unconnected-(U8-Pad1) -> /SPI_CS_N
- U8 pad 2: unconnected-(U8-Pad2) -> /SPI_SCK
- U8 pad 3: unconnected-(U8-Pad3) -> /SPI_MOSI
Changed lines of the file:
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@@
 			(size 0.2794 1.3589)
 			(layers "F.Cu" "F.Mask" "F.Paste")
-			(net "+3.3V")
+			(net "data_oe_n")
 			(pinfunction "PR9A_58")
 			(pintype "unspecified")
@@
 			(size 0.2794 1.3589)
 			(layers "F.Cu" "F.Mask" "F.Paste")
-			(net "unconnected-(U5-PT10B-Pad96)")
+			(net "/SPI_MOSI")
 			(pinfunction "PT10B_96")
 			(pintype "unspecified")
@@
 			(size 0.2794 1.3589)
 			(layers "F.Cu" "F.Mask" "F.Paste")
-			(net "unconnected-(U5-PT10A-Pad97)")
+			(net "/SPI_CS_N")
 			(pinfunction "PT10A_97")
 			(pintype "unspecified")
@@
 			(size 0.2794 1.3589)
 			(layers "F.Cu" "F.Mask" "F.Paste")
-			(net "unconnected-(U5-PT9B-Pad98)")
+			(net "/SPI_SCK")
 			(pinfunction "PT9B_98")
 			(pintype "unspecified")
@@
 			(size 0.2794 1.3589)
 			(layers "F.Cu" "F.Mask" "F.Paste")
-			(net "unconnected-(U5-PT9A-Pad99)")
+			(net "/SPI_MISO")
 			(pinfunction "PT9A_99")
 			(pintype "unspecified")
@@
 		)
 	)
+	(footprint "Resistor_SMD:R_0603_1608Metric_Pad0.98x0.95mm_HandSolder"
+		(layer "F.Cu")
+		(at 161.215 49.555)
+		(descr "Resistor SMD 0603 (1608 Metric), square (rectangular) end terminal, IPC-7351 nominal with elongated pad for handsoldering. (Body size source: IPC-SM-782 page 72, https://www.pcb-3d.com/wordpress/wp-content/uploads/ipc-sm-782a_amendment_1_and_2.pdf)")
+		(tags "resistor handsolder")
+		(property "Reference" "R3"
+			(at 0 -1.43 0)
+			(layer "F.SilkS")
+			(effects
+				(font
+					(size 1 1)
+					(thickness 0.15)
+				)
+			)
+		)
+		(property "Value" "10K"
+			(at 0 1.43 0)
+			(layer "F.Fab")
+			(effects
+				(font
+					(size 1 1)
+					(thickness 0.15)
+				)
+			)
+		)
+		(property "Datasheet" ""
+			(at 0 0 0)
+			(layer "F.Fab")
+			(hide yes)
+			(effects
+				(font
+					(size 1.27 1.27)
+				)
+			)
+		)
+		(property "Description" "Resistor"
+			(at 0 0 0)
+			(layer "F.Fab")
+			(hide yes)
+			(effects
+				(font
+					(size 1.27 1.27)
+				)
+			)
+		)
+		(property "KiLib_Generator" "SMD_2terminal_chip_molded"
+			(at 0 0 0)
+			(layer "F.SilkS")
+			(hide yes)
+			(effects
+				(font
+					(size 1 1)
+					(thickness 0.15)
+				)
+			)
+		)
+		(property ki_fp_filters "R_*")
+		(sheetname "/")
+		(sheetfile "cartridge.kicad_sch")
+		(units
+			(unit
+				(name "A")
+				(pins "1" "2")
+			)
+		)
+		(attr smd)
+		(duplicate_pad_numbers_are_jumpers no)
+		(fp_line
+			(start -0.254724 -0.5225)
+			(end 0.254724 -0.5225)
+			(stroke
+				(width 0.12)
+				(type solid)
+			)
+			(layer "F.SilkS")
+		)
+		(fp_line
+			(start -0.254724 0.5225)
+			(end 0.254724 0.5225)
+			(stroke
+				(width 0.12)
+				(type solid)
+			)
+			(layer "F.SilkS")
+		)
+		(fp_rect
+			(start -1.65 -0.73)
+			(end 1.65 0.73)
+			(stroke
+				(width 0.05)
+				(type solid)
+			)
+			(fill no)
+			(layer "F.CrtYd")
+		)
+		(fp_rect
+			(start -0.8 -0.4125)
+			(end 0.8 0.4125)
+			(stroke
+				(width 0.1)
+				(type solid)
+			)
+			(fill no)
+			(layer "F.Fab")
+		)
+		(fp_text user "${REFERENCE}"
+			(at 0 0 0)
+			(layer "F.Fab")
+			(effects
+				(font
+					(size 0.4 0.4)
+					(thickness 0.06)
+				)
+			)
+		)
+		(pad "1" smd roundrect
+			(at -0.9125 0)
+			(size 0.975 0.95)
+			(layers "F.Cu" "F.Mask" "F.Paste")
+			(roundrect_rratio 0.25)
+			(net "data_oe_n")
+			(pintype "passive")
+		)
+		(pad "2" smd roundrect
+			(at 0.9125 0)
+			(size 0.975 0.95)
+			(layers "F.Cu" "F.Mask" "F.Paste")
+			(roundrect_rratio 0.25)
+			(net "+3.3V")
+			(pintype "passive")
+		)
+		(embedded_fonts no)
+		(model "${KICAD10_3DMODEL_DIR}/Resistor_SMD.3dshapes/R_0603_1608Metric.step"
+			(offset
+				(xyz 0 0 0)
+			)
+			(scale
+				(xyz 1 1 1)
+			)
+			(rotate
+				(xyz 0 0 0)
+			)
+		)
+	)
 	(footprint "RP2040-Zero:RP2040-Zero"
 		(layer "F.Cu")
@@
 			(layers "*.Cu" "*.Mask")
 			(remove_unused_layers no)
-			(net "unconnected-(U8-Pad0)")
+			(net "/SPI_MISO")
 			(pinfunction "0_0")
 			(pintype "bidirectional")
@@
 			(layers "*.Cu" "*.Mask")
 			(remove_unused_layers no)
-			(net "unconnected-(U8-Pad1)")
+			(net "/SPI_CS_N")
 			(pinfunction "1_1")
 			(pintype "bidirectional")
@@
 			(layers "*.Cu" "*.Mask")
 			(remove_unused_layers no)
-			(net "unconnected-(U8-Pad2)")
+			(net "/SPI_SCK")
 			(pinfunction "2_2")
 			(pintype "bidirectional")
@@
 			(layers "*.Cu" "*.Mask")
 			(remove_unused_layers no)
-			(net "unconnected-(U8-Pad3)")
+			(net "/SPI_MOSI")
 			(pinfunction "3_3")
 			(pintype "bidirectional")
@@
 			(size 1.6764 0.3556)
 			(layers "F.Cu" "F.Mask" "F.Paste")
-			(net "Net-(U3-*OE)")
+			(net "data_oe_n")
 			(pinfunction "*OE_22")
 			(pintype "input")

Commit message: Update schematics
Connections:
- net /SPI_CS_N renamed SPI_CS_N
- net /SPI_MISO renamed SPI_MISO
- net /SPI_MOSI renamed SPI_MOSI
- net /SPI_SCK renamed SPI_SCK
Changed lines of the file:
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@@
 			(size 0.2794 1.3589)
 			(layers "F.Cu" "F.Mask" "F.Paste")
-			(net "/SPI_MOSI")
+			(net "SPI_MOSI")
 			(pinfunction "PT10B_96")
 			(pintype "unspecified")
@@
 			(size 0.2794 1.3589)
 			(layers "F.Cu" "F.Mask" "F.Paste")
-			(net "/SPI_CS_N")
+			(net "SPI_CS_N")
 			(pinfunction "PT10A_97")
 			(pintype "unspecified")
@@
 			(size 0.2794 1.3589)
 			(layers "F.Cu" "F.Mask" "F.Paste")
-			(net "/SPI_SCK")
+			(net "SPI_SCK")
 			(pinfunction "PT9B_98")
 			(pintype "unspecified")
@@
 			(size 0.2794 1.3589)
 			(layers "F.Cu" "F.Mask" "F.Paste")
-			(net "/SPI_MISO")
+			(net "SPI_MISO")
 			(pinfunction "PT9A_99")
 			(pintype "unspecified")
@@
 			(layers "*.Cu" "*.Mask")
 			(remove_unused_layers no)
-			(net "/SPI_MISO")
+			(net "SPI_MISO")
 			(pinfunction "0_0")
 			(pintype "bidirectional")
@@
 			(layers "*.Cu" "*.Mask")
 			(remove_unused_layers no)
-			(net "/SPI_CS_N")
+			(net "SPI_CS_N")
 			(pinfunction "1_1")
 			(pintype "bidirectional")
@@
 			(layers "*.Cu" "*.Mask")
 			(remove_unused_layers no)
-			(net "/SPI_SCK")
+			(net "SPI_SCK")
 			(pinfunction "2_2")
 			(pintype "bidirectional")
@@
 			(layers "*.Cu" "*.Mask")
 			(remove_unused_layers no)
-			(net "/SPI_MOSI")
+			(net "SPI_MOSI")
 			(pinfunction "3_3")
 			(pintype "bidirectional")

Commit message: Update plan and schematics
Parts:
- added R10: 10K, Resistor_SMD:R_0603_1608Metric_Pad0.98x0.95mm_HandSolder, F.Cu at (177.2, 90.7)
- added R5: 10K, Resistor_SMD:R_0603_1608Metric_Pad0.98x0.95mm_HandSolder, F.Cu at (177.2, 78.2)
- added R6: 10K, Resistor_SMD:R_0603_1608Metric_Pad0.98x0.95mm_HandSolder, F.Cu at (177.2, 80.7)
- added R7: 10K, Resistor_SMD:R_0603_1608Metric_Pad0.98x0.95mm_HandSolder, F.Cu at (177.2, 83.2)
- added R8: 10K, Resistor_SMD:R_0603_1608Metric_Pad0.98x0.95mm_HandSolder, F.Cu at (177.2, 85.7)
- added R9: 10K, Resistor_SMD:R_0603_1608Metric_Pad0.98x0.95mm_HandSolder, F.Cu at (177.2, 88.2)
Connections:
- C10 pad 1: Net-(U7-VDD) -> +3.3V
- U1 pad 10: gb_a8 -> gb_a7
- U1 pad 3: gb_a1 -> gb_a0
- U1 pad 4: gb_a2 -> gb_a1
- U1 pad 5: gb_a3 -> gb_a2
- U1 pad 6: gb_a4 -> gb_a3
- U1 pad 7: gb_a5 -> gb_a4
- U1 pad 8: gb_a6 -> gb_a5
- U1 pad 9: gb_a7 -> gb_a6
- U5 pad 82: unconnected-(U5-PT15C-Pad82) -> fram_ce_n
- U5 pad 83: unconnected-(U5-PT15B-Pad83) -> fram_oe_n
- U5 pad 84: unconnected-(U5-PT15A-Pad84) -> fram_we_n
- U7 pad 1: unconnected-(U7-A11-Pad1) -> flash_a11
- U7 pad 10: unconnected-(U7-A16-Pad10) -> flash_a16
- U7 pad 11: unconnected-(U7-A14-Pad11) -> flash_a14
- U7 pad 12: unconnected-(U7-A12-Pad12) -> flash_a12
- U7 pad 13: unconnected-(U7-A7-Pad13) -> flash_a7
- U7 pad 14: unconnected-(U7-A6-Pad14) -> flash_a6
- U7 pad 15: unconnected-(U7-A5-Pad15) -> flash_a5
- U7 pad 16: unconnected-(U7-A4-Pad16) -> flash_a4
- U7 pad 17: unconnected-(U7-A3-Pad17) -> flash_a3
- U7 pad 18: unconnected-(U7-A2-Pad18) -> flash_a2
- U7 pad 19: unconnected-(U7-A1-Pad19) -> flash_a1
- U7 pad 2: unconnected-(U7-A9-Pad2) -> flash_a9
- U7 pad 20: unconnected-(U7-A0-Pad20) -> flash_a0
- U7 pad 21: unconnected-(U7-DQ0-Pad21) -> flash_d0
- U7 pad 22: unconnected-(U7-DQ1-Pad22) -> flash_d1
- U7 pad 23: unconnected-(U7-DQ2-Pad23) -> flash_d2
- U7 pad 25: unconnected-(U7-DQ3-Pad25) -> flash_d3
- U7 pad 26: unconnected-(U7-DQ4-Pad26) -> flash_d4
- U7 pad 27: unconnected-(U7-DQ5-Pad27) -> flash_d5
- U7 pad 28: unconnected-(U7-DQ6-Pad28) -> flash_d6
- U7 pad 29: unconnected-(U7-DQ7-Pad29) -> flash_d7
- U7 pad 3: unconnected-(U7-A8-Pad3) -> flash_a8
- U7 pad 30: unconnected-(U7-*CE1-Pad30) -> fram_ce_n
- U7 pad 31: unconnected-(U7-A10-Pad31) -> fram_a10
- U7 pad 32: unconnected-(U7-*OE-Pad32) -> fram_oe_n
- U7 pad 4: unconnected-(U7-A13-Pad4) -> flash_a13
- U7 pad 5: unconnected-(U7-*WE-Pad5) -> fram_we_n
- U7 pad 6: unconnected-(U7-CE2-Pad6) -> +3.3V
- U7 pad 7: unconnected-(U7-A15-Pad7) -> flash_a15
- U7 pad 8: Net-(U7-VDD) -> +3.3V

Commit message: update schematics
Parts:
- moved C6 38.6 mm to (171.6, 91.9)
- moved C8 38.1 mm to (140.8, 91.9)
- moved C9 37.6 mm to (145.2, 81.1), turned to -90 degrees
- moved C2 37.5 mm to (161.6, 91.9)
- moved C4 32.6 mm to (151.2, 91.9)
- moved R4 28.9 mm to (158.5, 81.3)
- moved C7 24.7 mm to (149.9, 79.2)
- moved C3 18.0 mm to (152.2, 74.7)
- moved C1 14.3 mm to (152.0, 65.7)
- moved R5 10.6 mm to (172.8, 68.5), turned to 180 degrees
Routing:
- net VCCB: track 0.00 -> 46.1 mm
- net +3.3V: track 0.00 -> 8.62 mm
- net data_dir: track 0.00 -> 2.63 mm
- net fram_ce_n: track 0.00 -> 2.35 mm

Commit message: Progress
Parts:
- added C21: 1uF / 10V X7R, Capacitor_SMD:C_0805_2012Metric_Pad1.18x1.45mm_HandSolder, F.Cu at (121.4, 102.0)
- added C22: 1uF / 10V X7R, Capacitor_SMD:C_0805_2012Metric_Pad1.18x1.45mm_HandSolder, F.Cu at (121.4, 105.0)
- added C23: 100nF / 10V, Capacitor_SMD:C_0603_1608Metric_Pad1.08x0.95mm_HandSolder, F.Cu at (116.8, 101.7)
- added C24: 47uF / 10V X5R, Capacitor_SMD:C_1210_3225Metric_Pad1.33x2.70mm_HandSolder, F.Cu at (126.8, 108.7)
- added C25: 10uF / 10V X7R, Capacitor_SMD:C_0805_2012Metric_Pad1.18x1.45mm_HandSolder, F.Cu at (121.4, 108.0)
- added C26: 100nF / 10V, Capacitor_SMD:C_0603_1608Metric_Pad1.08x0.95mm_HandSolder, F.Cu at (116.8, 104.2)
- added C27: 22uF / 10V tantalum, Capacitor_Tantalum_SMD:CP_EIA-3528-21_Kemet-B, F.Cu at (126.8, 113.0)
- added C28: 100nF / 10V, Capacitor_SMD:C_0603_1608Metric, F.Cu at (121.0, 110.8)
- added J1: GameBoy_GamePak_DMG-09, Connector_GameBoy:GameBoy_GamePak_DMG-09_P1.50mm_Edge, F.Cu at (80.8, 114.1)
- added R11: 10K, Resistor_SMD:R_0603_1608Metric_Pad0.98x0.95mm_HandSolder, F.Cu at (122.5, 96.7)
- added R12: 330k 1%, Resistor_SMD:R_0603_1608Metric_Pad0.98x0.95mm_HandSolder, F.Cu at (116.8, 106.8)
- added R13: 100k 1%, Resistor_SMD:R_0603_1608Metric_Pad0.98x0.95mm_HandSolder, F.Cu at (116.8, 109.3)
- added U10: AMS1117-3.3, Package_TO_SOT_SMD:SOT-89-3, F.Cu at (127.1, 103.6)
- added U9: TPS2116DRL, Package_TO_SOT_SMD:SOT-583-8, F.Cu at (116.4, 112.5)
- moved U8 119.4 mm to (66.7, 65.7)
- moved C2 96.5 mm to (65.5, 100.6), turned to 90 degrees
- moved U7 92.0 mm to (72.2, 86.1)
- moved C1 91.6 mm to (65.5, 95.9), turned to -90 degrees
- moved C3 79.6 mm to (75.5, 95.9), turned to -90 degrees
- moved C6 77.4 mm to (94.5, 98.4), turned to 90 degrees
- moved U2 76.4 mm to (70.5, 98.2)
- moved C4 76.2 mm to (75.5, 100.6), turned to 90 degrees
- moved U1 75.9 mm to (60.5, 98.2)
- moved U4 68.1 mm to (99.6, 98.2)
- moved U3 68.0 mm to (89.4, 98.2)
- moved U6 50.4 mm to (93.2, 65.2)
- moved U5 49.2 mm to (93.5, 82.5)
- moved C8 36.7 mm to (104.6, 98.4), turned to 90 degrees
Connections:
- U1 pad 10: gb_a7 -> gb_a0
- U1 pad 14: A7 -> A0
- U1 pad 15: A6 -> A1
- U1 pad 16: A5 -> A2
- U1 pad 17: A4 -> A3
- U1 pad 18: A3 -> A4
- U1 pad 19: A2 -> A5
- U1 pad 20: A1 -> A6
- U1 pad 21: A0 -> A7
- U1 pad 3: gb_a0 -> gb_a7
- U1 pad 4: gb_a1 -> gb_a6
- U1 pad 5: gb_a2 -> gb_a5
- U1 pad 6: gb_a3 -> gb_a4
- U1 pad 7: gb_a4 -> gb_a3
- U1 pad 8: gb_a5 -> gb_a2
- U1 pad 9: gb_a6 -> gb_a1
- U2 pad 10: gb_a15 -> gb_a8
- U2 pad 14: A15 -> A8
- U2 pad 15: A14 -> A9
- U2 pad 16: A13 -> A10
- U2 pad 17: A12 -> A11
- U2 pad 18: A11 -> A12
- U2 pad 19: A10 -> A13
- U2 pad 20: A9 -> A14
- U2 pad 21: A8 -> A15
- U2 pad 3: gb_a8 -> gb_a15
- U2 pad 4: gb_a9 -> gb_a14
- U2 pad 5: gb_a10 -> gb_a13
- U2 pad 6: gb_a11 -> gb_a12
- U2 pad 7: gb_a12 -> gb_a11
- U2 pad 8: gb_a13 -> gb_a10
- U2 pad 9: gb_a14 -> gb_a9
- U3 pad 10: gb_d7 -> gb_d0
- U3 pad 14: D7 -> D0
- U3 pad 15: D6 -> D1
- U3 pad 16: D5 -> D2
- U3 pad 17: D4 -> D3
- U3 pad 18: D3 -> D4
- U3 pad 19: D2 -> D5
- U3 pad 20: D1 -> D6
- U3 pad 21: D0 -> D7
- U3 pad 3: gb_d0 -> gb_d7
- U3 pad 4: gb_d1 -> gb_d6
- U3 pad 5: gb_d2 -> gb_d5
- U3 pad 6: gb_d3 -> gb_d4
- U3 pad 7: gb_d4 -> gb_d3
- U3 pad 8: gb_d5 -> gb_d2
- U3 pad 9: gb_d6 -> gb_d1
- U4 pad 17: GND -> VCCB
- U4 pad 7: GND -> gb_power_present
- U5 pad 85: unconnected-(U5-PT12D-Pad85) -> gb_power_present
- U7 pad 31: fram_a10 -> flash_a10
- U8 pad 3v3: +3.3V -> unconnected-(U8-Pad3v3)
Routing:
- net gb_wr_n: track 0.00 -> 56.3 mm
- net /WR: track 0.00 -> 46.4 mm, vias 0 -> 2
- net /RD: track 0.00 -> 44.4 mm, vias 0 -> 2
- net /CS: track 0.00 -> 40.5 mm, vias 0 -> 2
- net VCCB: track 46.1 -> 13.1 mm, vias 0 -> 4
- net gb_rd_n: track 0.00 -> 32.1 mm
- net gb_cs_n: track 0.00 -> 30.2 mm
- net gb_a8: track 0.00 -> 27.4 mm
- net gb_a9: track 0.00 -> 27.4 mm
- net gb_a11: track 0.00 -> 26.9 mm
- net gb_a13: track 0.00 -> 26.7 mm
- net gb_a15: track 0.00 -> 26.4 mm
- net A15: track 0.00 -> 23.2 mm, vias 0 -> 2
- net A12: track 0.00 -> 22.3 mm, vias 0 -> 2
- net A14: track 0.00 -> 21.6 mm, vias 0 -> 2
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- added copper zone on In2.Cu, net +3.3V
- added copper zone on In1.Cu, net GND
- added copper zone on In2.Cu, net VCCB
Other:
- board size 71.2 x 52.2 mm -> 51 x 60.7 mm
- copper layers 2 -> 4
