File: hardware/cartridge/cartridge.kicad_sch (KiCad schematic)
At the start: 37 parts, among them U1 SN74LVC8T245PWR, U2 SN74LVC8T245PWR, U3 SN74LVC8T245PWR, U4 SN74LVC8T245PWR, U5 LCMXO2-1200HC-4TG100C, U6 MX29LV320EBTI-70G, U7 FM28V100-TG, U8 RP2040-Zero

Commit message: add 2in1 fpga firmware (untested)
Parts:
- added R11: 10K, Resistor_SMD:R_0603_1608Metric_Pad0.98x0.95mm_HandSolder, symbol Device:R
Connections:
- net GND: now also R11.1; no longer U4.17 (B5), U4.7 (A5)
- net VCCB: now also U4.17 (B5)
- net gb_power_present: now reaches U5.85 (PT12D)
- net gb_power_present: now also U4.7 (A5), R11.2
Other:
- note added: "U4 B5 -> A5: детектор питания. R11 задаёт LOW при Hi-Z U4;"

Commit message: Power muxing prototype
Connections:
- net +3.3V: no longer U8.3v3
- no-connect marks 1 -> 2
Other:
- added sheet Power - TPS2116 + AMS1117 (power_mux.kicad_sch)
- note added: "3.3 V from on-board AMS1117 to cartridge"
- note added: "U8.3v3 isolated; USB powers RP2040 separately"
Changed lines of the file:
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@@
 		)
 	)
+	(text "3.3 V from on-board AMS1117 to cartridge"
+		(exclude_from_sim no)
+		(at 204.47 265.43 0)
+		(effects
+			(font
+				(size 1.27 1.27)
+			)
+		)
+	)
 	(text "Подтяжки 10 кОм к 3,3 В: память отключена при Hi-Z FPGA"
 		(exclude_from_sim no)
@@
 		)
 	)
+	(text "U8.3v3 isolated; USB powers RP2040 separately"
+		(exclude_from_sim no)
+		(at 209.55 273.05 0)
+		(effects
+			(font
+				(size 1.27 1.27)
+			)
+		)
+	)
 	(junction
 		(at 351.79 234.95)
@@
 		(at 185.42 52.07)
 	)
+	(no_connect
+		(at 367.03 82.55)
+	)
 	(wire
 		(pts
@@
 	(wire
 		(pts
+			(xy 124.46 265.43) (xy 144.78 265.43)
+		)
+		(stroke
+			(width 0)
+			(type default)
+		)
+	)
+	(wire
+		(pts
 			(xy 46.99 142.24) (xy 57.15 142.24)
 		)
@@
 	(wire
 		(pts
+			(xy 54.61 265.43) (xy 30.48 265.43)
+		)
+		(stroke
+			(width 0)
+			(type default)
+		)
+	)
+	(wire
+		(pts
+			(xy 54.61 273.05) (xy 30.48 273.05)
+		)
+		(stroke
+			(width 0)
+			(type default)
+		)
+	)
+	(wire
+		(pts
 			(xy 128.27 238.76) (xy 135.89 238.76)
 		)
@@
 	(wire
 		(pts
+			(xy 124.46 273.05) (xy 144.78 273.05)
+		)
+		(stroke
+			(width 0)
+			(type default)
+		)
+	)
+	(wire
+		(pts
 			(xy 24.13 246.38) (xy 57.15 246.38)
 		)
@@
 		)
 	)
+	(label "+3.3V"
+		(at 144.78 265.43 0)
+		(effects
+			(font
+				(size 1.27 1.27)
+			)
+			(justify left bottom)
+		)
+	)
+	(label "GND"
+		(at 144.78 273.05 0)
+		(effects
+			(font
+				(size 1.27 1.27)
+			)
+			(justify left bottom)
+		)
+	)
 	(label "gb_power_present"
 		(at 138.43 160.02 0)
@@
 		)
 	)
+	(label "+5V (USB)"
+		(at 30.48 273.05 0)
+		(effects
+			(font
+				(size 1.27 1.27)
+			)
+			(justify left bottom)
+		)
+	)
+	(label "VCCB"
+		(at 30.48 265.43 0)
+		(effects
+			(font
+				(size 1.27 1.27)
+			)
+			(justify left bottom)
+		)
+	)
 	(symbol
 		(lib_id "power:VSSA")
@@
 	)
 	(symbol
-		(lib_id "power:+3.3V")
-		(at 367.03 82.55 270)
-		(mirror x)
-		(unit 1)
-		(body_style 1)
-		(exclude_from_sim no)
-		(in_bom yes)
-		(on_board yes)
-		(in_pos_files yes)
-		(dnp no)
-		(property "Reference" "#PWR0306"
-			(at 363.22 82.55 0)
-			(hide yes)
-			(show_name no)
-			(do_not_autoplace no)
-			(effects
-				(font
-					(size 1.27 1.27)
-				)
-			)
-		)
-		(property "Value" "+3.3V"
-			(at 370.84 82.5499 90)
-			(show_name no)
-			(do_not_autoplace no)
-			(effects
-				(font
-					(size 1.27 1.27)
-				)
-				(justify left)
-			)
-		)
-		(property "Footprint" ""
-			(at 367.03 82.55 0)
-			(hide yes)
-			(show_name no)
-			(do_not_autoplace no)
-			(effects
-				(font
-					(size 1.27 1.27)
-				)
-			)
-		)
-		(property "Datasheet" ""
-			(at 367.03 82.55 0)
-			(hide yes)
-			(show_name no)
-			(do_not_autoplace no)
-			(effects
-				(font
-					(size 1.27 1.27)
-				)
-			)
-		)
-		(property "Description" "Power symbol creates a global label with name \"+3.3V\""
-			(at 367.03 82.55 0)
-			(hide yes)
-			(show_name no)
-			(do_not_autoplace no)
-			(effects
-				(font
-					(size 1.27 1.27)
-				)
-			)
-		)
-		(pin "1"
-		)
-		(instances
-			(project "cartridge"
-				(path "/2780facd-cffd-485a-aed1-c460c817db24"
-					(reference "#PWR0306")
-					(unit 1)
-				)
-			)
-		)
-	)
-	(symbol
 		(lib_id "power:VSSA")
 		(at 242.57 170.18 270)
@@
 				)
 			)
+		)
+	)
+	(sheet
+		(at 54.61 260.35)
+		(size 71.12 17.78)
+		(exclude_from_sim no)
+		(in_bom yes)
+		(on_board yes)
+		(dnp no)
+		(stroke
+			(width 0.254)
+			(type solid)
+		)
+		(fill
+			(color 0 0 0 0)
+		)
+		(property "Sheetname" "Power - TPS2116 + AMS1117"
+			(at 54.61 259.08 0)
+			(show_name no)
+			(do_not_autoplace no)
+			(effects
+				(font
+					(size 1.27 1.27)
+				)
+				(justify left bottom)
+			)
+		)
+		(property "Sheetfile" "power_mux.kicad_sch"
+			(at 54.61 279.4 0)
+			(show_name no)
+			(do_not_autoplace no)
+			(effects
+				(font
+					(size 1.27 1.27)
+				)
+				(justify left top)
+			)
+		)
+		(pin "GB_5V" input
+			(at 54.61 265.43 180)
+			(effects
+				(font
+					(size 1.27 1.27)
+				)
+				(justify left)
+			)
+		)
+		(pin "USB_5V" input
+			(at 54.61 273.05 180)
+			(effects
+				(font
+					(size 1.27 1.27)
+				)
+				(justify left)
+			)
+		)
+		(pin "CART_3V3" output
+			(at 125.73 265.43 0)
+			(effects
+				(font
+					(size 1.27 1.27)
+				)
+				(justify right)
+			)
+		)
+		(pin "GND" input
+			(at 125.73 273.05 0)
+			(effects
+				(font
+					(size 1.27 1.27)
+				)
+				(justify right)
+			)
+		)
+		(instances
+			(project "cartridge"
+				(path "/2780facd-cffd-485a-aed1-c460c817db24"
+					(page "2")
+				)
+			)

Commit message: Progress
Parts:
- added J1: GameBoy_GamePak_DMG-09, Connector_GameBoy:GameBoy_GamePak_DMG-09_P1.50mm_Edge, symbol kicad-gamepaks:GameBoy_GamePak_DMG-09
Connections:
- net /CS: now also J1.5 (~{CS})
- net /RD: now also J1.4 (~{RD})
- net /RES: now also J1.30 (~{RST})
- net /WR: now also J1.3 (~{WR})
- net A0: now also U1.14 (B8), J1.6 (A0); no longer U1.21 (B1)
- net A1: now also U1.15 (B7), J1.7 (A1); no longer U1.20 (B2)
- net A10: now also U2.16 (B6), J1.16 (A10); no longer U2.19 (B3)
- net A11: now also U2.17 (B5), J1.17 (A11); no longer U2.18 (B4)
- net A12: now also U2.18 (B4), J1.18 (A12); no longer U2.17 (B5)
- net A13: now also U2.19 (B3), J1.19 (A13); no longer U2.16 (B6)
- net A14: now also U2.20 (B2), J1.20 (A14); no longer U2.15 (B7)
- net A15: now also U2.21 (B1), J1.21 (A15); no longer U2.14 (B8)
- net A2: now also U1.16 (B6), J1.8 (A2); no longer U1.19 (B3)
- net A3: now also U1.17 (B5), J1.9 (A3); no longer U1.18 (B4)
- net A4: now also U1.18 (B4), J1.10 (A4); no longer U1.17 (B5)
- net A5: now also U1.19 (B3), J1.11 (A5); no longer U1.16 (B6)
- net A6: now also U1.20 (B2), J1.12 (A6); no longer U1.15 (B7)
- net A7: now also U1.21 (B1), J1.13 (A7); no longer U1.14 (B8)
- net A8: now also U2.14 (B8), J1.14 (A8); no longer U2.21 (B1)
- net A9: now also U2.15 (B7), J1.15 (A9); no longer U2.20 (B2)
- net D0: now also U3.14 (B8), J1.22 (D0); no longer U3.21 (B1)
- net D1: now also U3.15 (B7), J1.23 (D1); no longer U3.20 (B2)
- net D2: now also U3.16 (B6), J1.24 (D2); no longer U3.19 (B3)
- net D3: now also U3.17 (B5), J1.25 (D3); no longer U3.18 (B4)
- net D4: now also U3.18 (B4), J1.26 (D4); no longer U3.17 (B5)
- net D5: now also U3.19 (B3), J1.27 (D5); no longer U3.16 (B6)
- net D6: now also U3.20 (B2), J1.28 (D6); no longer U3.15 (B7)
- net D7: now also U3.21 (B1), J1.29 (D7); no longer U3.14 (B8)
- net GND: now also J1.32 (GND)
- net VCCB: now also J1.1 (VCC)
- net gb_a0: now also U1.10 (A8); no longer U1.3 (A1)
- net gb_a1: now also U1.9 (A7); no longer U1.4 (A2)
- net gb_a10: now also U2.8 (A6); no longer U2.5 (A3)
- net gb_a11: now also U2.7 (A5); no longer U2.6 (A4)
- net gb_a12: now also U2.6 (A4); no longer U2.7 (A5)
- net gb_a13: now also U2.5 (A3); no longer U2.8 (A6)
- net gb_a14: now also U2.4 (A2); no longer U2.9 (A7)
- net gb_a15: now also U2.3 (A1); no longer U2.10 (A8)
- net gb_a2: now also U1.8 (A6); no longer U1.5 (A3)
- net gb_a3: now also U1.7 (A5); no longer U1.6 (A4)
- net gb_a4: now also U1.6 (A4); no longer U1.7 (A5)
- net gb_a5: now also U1.5 (A3); no longer U1.8 (A6)
- net gb_a6: now also U1.4 (A2); no longer U1.9 (A7)
- net gb_a7: now also U1.3 (A1); no longer U1.10 (A8)
- net gb_a8: now also U2.10 (A8); no longer U2.3 (A1)
- net gb_a9: now also U2.9 (A7); no longer U2.4 (A2)
- net gb_d0: now also U3.10 (A8); no longer U3.3 (A1)
- net gb_d1: now also U3.9 (A7); no longer U3.4 (A2)
- net gb_d2: now also U3.8 (A6); no longer U3.5 (A3)
- net gb_d3: now also U3.7 (A5); no longer U3.6 (A4)
- net gb_d4: now also U3.6 (A4); no longer U3.7 (A5)
- net gb_d5: now also U3.5 (A3); no longer U3.8 (A6)
- net gb_d6: now also U3.4 (A2); no longer U3.9 (A7)
- net gb_d7: now also U3.3 (A1); no longer U3.10 (A8)
